File: SBC6309Ram.kicad_pcb (KiCad board)
At the start: 2 copper layers, 49.4 x 40.8 mm, 7 parts, among them J1 Address, J2 Device, J3 Clock, J4 Power, J5 Data, U1 W24512AK, U6 GAL16V8

Commit message: minor revision
Parts:
- added C1: 100nF, Capacitor_SMD:C_0805_2012Metric, F.Cu at (99.5, 81.7)
- added C2: 100nF, Capacitor_SMD:C_0805_2012Metric, F.Cu at (141.9, 109.2)
Routing:
- net GND: track 57.5 -> 0.00 mm, vias 35 -> 41
- net /R/~{W}: track 74.0 -> 68.8 mm
- net +5V: track 97.0 -> 100.0 mm
- net /CS2: track 60.9 -> 61.9 mm
- net /S3: track 17.2 -> 17.7 mm
- net /D6: track 52.0 -> 51.5 mm
