File: SBC6309Ram.kicad_sch (KiCad schematic)
At the start: 7 parts, among them J1 Address, J2 Device, J3 Clock, J4 Power, J5 Data, U1 W24512AK, U6 GAL16V8

Commit message: minor revision
Parts:
- added C1, C2: 100nF, Capacitor_SMD:C_0805_2012Metric, symbol Device:C_Small
Connections:
- net +5V: now also C1.1, C2.1
- net GND: now also C1.2, C2.2
